File: AppleII-Disk-Clacker/AppleII-Disk-Clacker.kicad_sch (KiCad schematic)
At the start: 11 parts, among them J1 Conn_02x10_Odd_Even, J2 Conn_02x10_Odd_Even, K1 SANYOU_SRD_Form_C, Q1 2N3904, U1 ATtiny13A-P

Commit message: Add a README
Parts:
- C1: MfrPartNo A104K15X7RF5TAA -> A104K15X7RF5TAA
- K1: MouserPartNo 523-AWHSH105D00G -> 523-AWHSH105D00G
- Q1: Mfr Diotec Semiconductor -> Diotec Semiconductor; MfrPartNo 2N3904 -> 2N3904; MouserPartNo 637-2N3904 -> 637-2N3904
- R1: Mfr KOA Speer -> KOA Speer; MfrPartNo MF1/4LCT52R222J -> MF1/4LCT52R222J
Changed lines of the file:
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@@
 				)
 				(justify left)
+				(hide yes)
 			)
 		)
@@
 			)
 		)
-		(property "MouserPartNo" " 523-AWHSH105D00G"
+		(property "MouserPartNo" "523-AWHSH105D00G"
 			(at 222.25 91.44 0)
 			(effects
@@
 			)
 		)
-		(property "Mfr" " Diotec Semiconductor"
+		(property "Mfr" "Diotec Semiconductor"
 			(at 214.63 109.22 0)
 			(effects
@@
 			)
 		)
-		(property "MfrPartNo" " 2N3904"
+		(property "MfrPartNo" "2N3904"
 			(at 214.63 109.22 0)
 			(effects
@@
 			)
 		)
-		(property "MouserPartNo" " 637-2N3904"
+		(property "MouserPartNo" "637-2N3904"
 			(at 214.63 109.22 0)
 			(effects
@@
 			)
 		)
-		(property "MfrPartNo" " A104K15X7RF5TAA"
+		(property "MfrPartNo" "A104K15X7RF5TAA"
 			(at 118.11 90.17 0)
 			(effects
@@
 			)
 		)
-		(property "Mfr" " KOA Speer"
+		(property "Mfr" "KOA Speer"
 			(at 203.2 109.22 90)
 			(effects
@@
 			)
 		)
-		(property "MfrPartNo" " MF1/4LCT52R222J"
+		(property "MfrPartNo" "MF1/4LCT52R222J"
 			(at 203.2 109.22 90)
 			(effects
